File: PCB/TrlPad.kicad_pcb (KiCad board)
At the start: 2 copper layers, 98.1 x 54.8 mm, 22 parts, among them SW1 SW_Push, SW2 SW_Push, SW3 SW_Push, SW4 SW_Push, SW5 RotaryEncoder_Switch, U1 XIAO-nRF52840-SMD, U2 128x32_OLED_S

Commit message: Updated BOM + fixed PCB
Parts:
- removed C1, C2: 10nF, Capacitor_SMD:C_0603_1608Metric_Pad1.08x0.95mm_HandSolder
- removed R3, R4, R5, R8: 10K, Resistor_SMD:R_0603_1608Metric_Pad0.98x0.95mm_HandSolder
Connections:
- SW5 pad A: Net-(R3-Pad1) -> /ENC_A
- SW5 pad B: Net-(R4-Pad2) -> /ENC_B
Routing:
- net Net-(R4-Pad2): track 40.6 -> 0.00 mm, vias 2 -> 0
- net VCC: track 77.4 -> 45.0 mm
- net Net-(R3-Pad1): track 21.4 -> 0.00 mm
- net /ENC_B: track 44.6 -> 38.9 mm, vias 2 -> 0
- net /ENC_A: track 31.0 -> 35.9 mm
- net /ROW 1: track 98.2 -> 97.0 mm
